Commit message: fix rotation axis & add rover blender model

File: src/mecanum_model/urdf/s1-based-rover.urdf.xacro (robot description, xacro)
@@ -15,5 +15,5 @@
     <visual>
       <geometry>
-        <mesh filename="package://urdf_tutorial/meshes/new/chassis.stl" scale="0.001 0.001 0.001"/>
+        <mesh filename="package://mecanum_model/meshes/chassis.stl" scale="0.001 0.001 0.001"/>
        </geometry>
        <material name="black" />
@@ -28,5 +28,5 @@
     <visual>
       <geometry>
-        <mesh filename="package://urdf_tutorial/meshes/new/sprayer_assembly.stl" scale="0.001 0.001 0.001"/>
+        <mesh filename="package://mecanum_model/meshes/sprayer_assembly.stl" scale="0.001 0.001 0.001"/>
        </geometry>
        <material name="light_grey" />
@@ -35,5 +35,5 @@
   <joint name="wheel1_shaft_joint" type="continuous">
      <origin xyz="-0.065 0.1 0.0" rpy="0 0 0" />
-      <axis xyz="0 1 0"/>
+      <axis xyz="1 0 0"/>
      <parent link="base_link"/>
      <child link="wheel1_shaft" />
@@ -43,12 +43,12 @@
      <origin xyz="0 0 0.0" rpy="0 0 0" />
      <geometry>
-       <mesh filename="package://urdf_tutorial/meshes/new/wheel_shaft.stl" scale="0.001 0.001 0.001"/>
-     </geometry>
-     <material name="black" />
-   </visual>
-   <collision>
-     <origin xyz="0 0 0.0"/>
-     <geometry>
-       <mesh filename="package://urdf_tutorial/meshes/new/wheel_shaft.stl" scale="0.001 0.001 0.001"/>
+       <mesh filename="package://mecanum_model/meshes/wheel_shaft_min.stl" scale="0.001 0.001 0.001"/>
+     </geometry>
+     <material name="black" />
+   </visual>
+   <collision>
+     <origin xyz="0 0 0.0"/>
+     <geometry>
+       <mesh filename="package://mecanum_model/meshes/wheel_shaft_min.stl" scale="0.001 0.001 0.001"/>
      </geometry>
    </collision>
@@ -71,5 +71,5 @@
       <origin xyz="0 0 0" rpy="0 0 0"/>
       <geometry>
-      	<mesh filename="package://urdf_tutorial/meshes/new/wheel_cw.stl" scale="0.001 0.001 0.001"/>
+      	<mesh filename="package://mecanum_model/meshes/wheel_cw.stl" scale="0.001 0.001 0.001"/>
 	     </geometry>
        <material name="light_grey" />
@@ -93,5 +93,5 @@
     <joint name="wheel2_shaft_joint" type="continuous">
      <origin xyz="0.065 0.1 0.0" rpy="0 0 0" />
-      <axis xyz="0 1 0"/>
+      <axis xyz="1 0 0"/>
      <parent link="base_link"/>
      <child link="wheel2_shaft" />
@@ -101,12 +101,12 @@
      <origin xyz="0 0 0.0" rpy="0 0 0" />
      <geometry>
-       <mesh filename="package://urdf_tutorial/meshes/new/wheel_shaft_max.stl" scale="0.001 0.001 0.001"/>
-     </geometry>
-     <material name="black" />
-   </visual>
-   <collision>
-     <origin xyz="0 0 0.0"/>
-     <geometry>
-       <mesh filename="package://urdf_tutorial/meshes/new/wheel_shaft_max.stl" scale="0.001 0.001 0.001"/>
+       <mesh filename="package://mecanum_model/meshes/wheel_shaft_max.stl" scale="0.001 0.001 0.001"/>
+     </geometry>
+     <material name="black" />
+   </visual>
+   <collision>
+     <origin xyz="0 0 0.0"/>
+     <geometry>
+       <mesh filename="package://mecanum_model/meshes/wheel_shaft_max.stl" scale="0.001 0.001 0.001"/>
      </geometry>
    </collision>
@@ -129,5 +129,5 @@
       <origin xyz="0 0 0" rpy="0 0 0"/>
       <geometry>
-      	<mesh filename="package://urdf_tutorial/meshes/new/wheel_ccw.stl" scale="0.001 0.001 0.001"/>
+      	<mesh filename="package://mecanum_model/meshes/wheel_ccw.stl" scale="0.001 0.001 0.001"/>
 	     </geometry>
        <material name="light_grey" />
@@ -151,5 +151,5 @@
    <joint name="wheel3_shaft_joint" type="continuous">
      <origin xyz="0.065 -0.1 0.0" rpy="0 0 0" />
-      <axis xyz="0 1 0"/>
+      <axis xyz="1 0 0"/>
      <parent link="base_link"/>
      <child link="wheel3_shaft" />
@@ -159,12 +159,12 @@
      <origin xyz="0 0 0.0" rpy="0 0 0" />
      <geometry>
-       <mesh filename="package://urdf_tutorial/meshes/new/wheel_shaft_max.stl" scale="0.001 0.001 0.001"/>
-     </geometry>
-     <material name="black" />
-   </visual>
-   <collision>
-     <origin xyz="0 0 0.0"/>
-     <geometry>
-       <mesh filename="package://urdf_tutorial/meshes/new/wheel_shaft_max.stl" scale="0.001 0.001 0.001"/>
+       <mesh filename="package://mecanum_model/meshes/wheel_shaft_max.stl" scale="0.001 0.001 0.001"/>
+     </geometry>
+     <material name="black" />
+   </visual>
+   <collision>
+     <origin xyz="0 0 0.0"/>
+     <geometry>
+       <mesh filename="package://mecanum_model/meshes/wheel_shaft_max.stl" scale="0.001 0.001 0.001"/>
      </geometry>
    </collision>
@@ -187,5 +187,5 @@
       <origin xyz="0 0 0" rpy="0 0 0"/>
       <geometry>
-      	<mesh filename="package://urdf_tutorial/meshes/new/wheel_cw.stl" scale="0.001 0.001 0.001"/>
+      	<mesh filename="package://mecanum_model/meshes/wheel_cw.stl" scale="0.001 0.001 0.001"/>
 	     </geometry>
        <material name="light_grey" />
@@ -209,5 +209,5 @@
    <joint name="wheel4_shaft_joint" type="continuous">
      <origin xyz="-0.065 -0.1 0.0" rpy="0 0 0" />
-      <axis xyz="0 1 0"/>
+      <axis xyz="1 0 0"/>
      <parent link="base_link"/>
      <child link="wheel4_shaft" />
@@ -217,12 +217,12 @@
      <origin xyz="0 0 0.0" rpy="0 0 0" />
      <geometry>
-       <mesh filename="package://urdf_tutorial/meshes/new/wheel_shaft_min.stl" scale="0.001 0.001 0.001"/>
-     </geometry>
-     <material name="black" />
-   </visual>
-   <collision>
-     <origin xyz="0 0 0.0"/>
-     <geometry>
-       <mesh filename="package://urdf_tutorial/meshes/new/wheel_shaft_min.stl" scale="0.001 0.001 0.001"/>
+       <mesh filename="package://mecanum_model/meshes/wheel_shaft_min.stl" scale="0.001 0.001 0.001"/>
+     </geometry>
+     <material name="black" />
+   </visual>
+   <collision>
+     <origin xyz="0 0 0.0"/>
+     <geometry>
+       <mesh filename="package://mecanum_model/meshes/wheel_shaft_min.stl" scale="0.001 0.001 0.001"/>
      </geometry>
    </collision>
@@ -245,5 +245,5 @@
       <origin xyz="0 0 0" rpy="0 0 0"/>
       <geometry>
-      	<mesh filename="package://urdf_tutorial/meshes/new/wheel_ccw.stl" scale="0.001 0.001 0.001"/>
+      	<mesh filename="package://mecanum_model/meshes/wheel_ccw.stl" scale="0.001 0.001 0.001"/>
 	     </geometry>
        <material name="light_grey" />

Commit message: working in gazebo, work more on model

File: src/mecanum_model/urdf/s1-based-rover.urdf.xacro (robot description, xacro)
@@ -6,21 +6,61 @@
   <material name="black"><color rgba="0.15 0.15 0.15 1.0" /></material>
   <material name="light_grey"><color rgba="0.4 0.4 0.4 1.0" /></material>
-  <link name="base_footprint"></link>
-  <joint name="base_link_joint" type="fixed">
+   <xacro:macro name="box_inertia" params="m w h d">
+    <inertial>
+      <origin xyz="0 0 0" rpy="${pi/2} 0 ${pi/2}"/>
+      <mass value="${m}"/>
+      <inertia ixx="${(m/12) * (h*h + d*d)}" ixy="0.0" ixz="0.0" iyy="${(m/12) * (w*w + d*d)}" iyz="0.0" izz="${(m/12) * (w*w + h*h)}"/>
+    </inertial>
+  </xacro:macro>
+  <xacro:macro name="cylinder_inertia" params="m r h">
+    <inertial>
+      <origin xyz="0 0 0" rpy="${pi/2} 0 0" />
+      <mass value="${m}"/>
+      <inertia ixx="${(m/12) * (3*r*r + h*h)}" ixy = "0" ixz = "0" iyy="${(m/12) * (3*r*r + h*h)}" iyz = "0" izz="${(m/2) * (r*r)}"/>
+    </inertial>
+  </xacro:macro>
+  <xacro:macro name="sphere_inertia" params="m r">
+    <inertial>
+      <mass value="${m}"/>
+      <inertia ixx="${(2/5) * m * (r*r)}" ixy="0.0" ixz="0.0" iyy="${(2/5) * m * (r*r)}" iyz="0.0" izz="${(2/5) * m * (r*r)}"/>
+    </inertial>
+  </xacro:macro>
+  <xacro:include filename="$(find mecanum_model)/urdf/s1-based-rover.gazebo" />
+  <link name="world"></link>
+  <joint name="fixed" type="fixed">
+    <parent link="world"/>
+    <child link="base_footprint"/>
+  </joint>
+  <link name="base_footprint">
+    <collision>
+      <origin rpy="0 0 0" xyz="0 0 0"/>
+      <geometry>
+	      <box size="${244.865616 * 0.001} ${302.041534 * 0.001} ${102.041229 * 0.001}"/>
+      </geometry>
+    </collision>
+  </link>
+  <joint name="chassis_joint" type="fixed">
     <origin xyz="0 0 0.0" rpy="0 0 0" />
     <parent link="base_footprint"/>
-    <child link="base_link" />
- </joint>
-  <link name="base_link">
-    <visual>
-      <geometry>
-        <mesh filename="package://mecanum_model/meshes/chassis.stl" scale="0.001 0.001 0.001"/>
+    <child link="chassis" />
+ </joint>
+  <link name="chassis">
+    <visual>
+      <geometry>
+        <mesh filename="$(find mecanum_model)/meshes/chassis.stl" scale="0.001 0.001 0.001"/>
        </geometry>
        <material name="black" />
     </visual>
+    <collision>
+      <origin rpy="0 0 0" xyz="0 0 0"/>
+      <geometry>
+	      <box size="${148.399536 * 0.001} ${252.206665 * 0.001} ${55.450001 * 0.001}"/>
+      </geometry>
+    </collision>
+    <xacro:box_inertia m="1.0" w="${148.399536 * 0.001}" d="${252.206665 * 0.001}" h="${55.450001 * 0.001}"/>
   </link>
   <joint name="sprayer_joint" type="fixed">
    <origin xyz="-0.003 -0.14 0.005" rpy="0 0 0" />
-   <parent link="base_link"/>
+   <parent link="chassis"/>
    <child link="sprayer_assembly" />
  </joint>
@@ -28,13 +68,20 @@
     <visual>
       <geometry>
-        <mesh filename="package://mecanum_model/meshes/sprayer_assembly.stl" scale="0.001 0.001 0.001"/>
+        <mesh filename="$(find mecanum_model)/meshes/sprayer_assembly.stl" scale="0.001 0.001 0.001"/>
        </geometry>
        <material name="light_grey" />
     </visual>
+    <collision>
+      <origin rpy="0 0 0" xyz="0 0 0"/>
+      <geometry>
+        <box size="${144.179398 * 0.001} ${69.498428 * 0.001} ${96.728165 * 0.001}"/>
+      </geometry>
+    </collision>
+    <xacro:box_inertia m="1.0" w="${144.179398 * 0.001}" d="${69.498428 * 0.001}" h="${96.728165 * 0.001}"/>
   </link>
   <joint name="wheel1_shaft_joint" type="continuous">
      <origin xyz="-0.065 0.1 0.0" rpy="0 0 0" />
       <axis xyz="1 0 0"/>
-     <parent link="base_link"/>
+     <parent link="chassis"/>
      <child link="wheel1_shaft" />
   </joint>
@@ -43,22 +90,15 @@
      <origin xyz="0 0 0.0" rpy="0 0 0" />
      <geometry>
-       <mesh filename="package://mecanum_model/meshes/wheel_shaft_min.stl" scale="0.001 0.001 0.001"/>
+       <mesh filename="$(find mecanum_model)/meshes/wheel_shaft_min.stl" scale="0.001 0.001 0.001"/>
      </geometry>
      <material name="black" />
    </visual>
    <collision>
-     <origin xyz="0 0 0.0"/>
-     <geometry>
-       <mesh filename="package://mecanum_model/meshes/wheel_shaft_min.stl" scale="0.001 0.001 0.001"/>
-     </geometry>
-   </collision>
-   <inertial>
-     <origin xyz="0 0 0" rpy="0 0 0"/>
-     <mass value="0.055"/>
-     <inertia
-       ixx="0.000021370" ixy="0" ixz="0"
-       iyy="0.000009966" iyz="0"
-       izz="0.000021370"/>
-   </inertial>
+      <origin rpy="0 0 0" xyz="0 0 0"/>
+      <geometry>
+        <box size="${32.400002 * 0.001} ${37.585724 * 0.001} ${37.599998 * 0.001}"/>
+      </geometry>
+    </collision>
+    <xacro:box_inertia m="1.0" w="${32.400002 * 0.001}" d="${37.585724 * 0.001}" h="${37.599998 * 0.001}"/>
  </link>
  <joint name="wheel1_wheel_joint" type="fixed">
@@ -71,28 +111,20 @@
       <origin xyz="0 0 0" rpy="0 0 0"/>
       <geometry>
-      	<mesh filename="package://mecanum_model/meshes/wheel_cw.stl" scale="0.001 0.001 0.001"/>
-	     </geometry>
-       <material name="light_grey" />
-    </visual>
-    <collision>
-      <origin xyz="0 0 0" rpy="0 0 0"/>
-      <geometry>
-        <cylinder radius="${wheel_radius}" length="${wheel_width}"/>
-      </geometry>
-    </collision>
-    <inertial>
-      <origin xyz="0 0 0.0" rpy="0 0 0"/>
-      <mass value="0.3844"/>
-      <!-- Inertia based on cylinder -->
-      <inertia
-        ixx="0.000324824" ixy="0" ixz="0"
-        iyy="0.000480000" iyz="0"
-        izz="0.000324824"/>
-    </inertial>
+      	<mesh filename="$(find mecanum_model)/meshes/wheel_cw.stl" scale="0.001 0.001 0.001"/>
+	     </geometry>
+       <material name="light_grey" />
+    </visual>
+     <collision>
+      <origin rpy="0 0 0" xyz="0 0 0"/>
+      <geometry>
+        <box size="${10  * 0.001} ${10* 0.001} ${102.040993 * 0.001}"/>
+      </geometry>
+    </collision>
+    <xacro:box_inertia m="1.0" w="${45.538025 * 0.001}" d="${102.041016 * 0.001}" h="${102.040993 * 0.001}"/>
   </link>
     <joint name="wheel2_shaft_joint" type="continuous">
      <origin xyz="0.065 0.1 0.0" rpy="0 0 0" />
       <axis xyz="1 0 0"/>
-     <parent link="base_link"/>
+     <parent link="chassis"/>
      <child link="wheel2_shaft" />
   </joint>
@@ -101,22 +133,15 @@
      <origin xyz="0 0 0.0" rpy="0 0 0" />
      <geometry>
-       <mesh filename="package://mecanum_model/meshes/wheel_shaft_max.stl" scale="0.001 0.001 0.001"/>
-     </geometry>
-     <material name="black" />
-   </visual>
-   <collision>
-     <origin xyz="0 0 0.0"/>
-     <geometry>
-       <mesh filename="package://mecanum_model/meshes/wheel_shaft_max.stl" scale="0.001 0.001 0.001"/>
-     </geometry>
-   </collision>
-   <inertial>
-     <origin xyz="0 0 0" rpy="0 0 0"/>
-     <mass value="0.055"/>
-     <inertia
-       ixx="0.000021370" ixy="0" ixz="0"
-       iyy="0.000009966" iyz="0"
-       izz="0.000021370"/>
-   </inertial>
+       <mesh filename="$(find mecanum_model)/meshes/wheel_shaft_max.stl" scale="0.001 0.001 0.001"/>
+     </geometry>
+     <material name="black" />
+   </visual>
+    <collision>
+      <origin rpy="0 0 0" xyz="0 0 0"/>
+      <geometry>
+        <box size="${32.400002 * 0.001} ${37.585724 * 0.001} ${37.599998 * 0.001}"/>
+      </geometry>
+    </collision>
+    <xacro:box_inertia m="1.0" w="${32.400002 * 0.001}" d="${37.585724 * 0.001}" h="${37.599998 * 0.001}"/>
  </link>
  <joint name="wheel2_wheel_joint" type="fixed">
@@ -129,28 +154,20 @@
       <origin xyz="0 0 0" rpy="0 0 0"/>
       <geometry>
-      	<mesh filename="package://mecanum_model/meshes/wheel_ccw.stl" scale="0.001 0.001 0.001"/>
-	     </geometry>
-       <material name="light_grey" />
-    </visual>
-    <collision>
-      <origin xyz="0 0 0" rpy="0 0 0"/>
-      <geometry>
-        <cylinder radius="${wheel_radius}" length="${wheel_width}"/>
-      </geometry>
-    </collision>
-    <inertial>
-      <origin xyz="0 0 0.0" rpy="0 0 0"/>
-      <mass value="0.3844"/>
-      <!-- Inertia based on cylinder -->
-      <inertia
-        ixx="0.000324824" ixy="0" ixz="0"
-        iyy="0.000480000" iyz="0"
-        izz="0.000324824"/>
-    </inertial>
+      	<mesh filename="$(find mecanum_model)/meshes/wheel_ccw.stl" scale="0.001 0.001 0.001"/>
+	     </geometry>
+       <material name="light_grey" />
+    </visual>
+    <collision>
+      <origin rpy="0 0 0" xyz="0 0 0"/>
+      <geometry>
+        <box size="${45.538025  * 0.001} ${102.041016 * 0.001} ${102.040993 * 0.001}"/>
+      </geometry>
+    </collision>
+    <xacro:box_inertia m="1.0" w="${45.538025 * 0.001}" d="${102.041016 * 0.001}" h="${102.040993 * 0.001}"/>
   </link>
    <joint name="wheel3_shaft_joint" type="continuous">
      <origin xyz="0.065 -0.1 0.0" rpy="0 0 0" />
-      <axis xyz="1 0 0"/>
-     <parent link="base_link"/>
+    <axis xyz="1 0 0"/>
+     <parent link="chassis"/>
      <child link="wheel3_shaft" />
   </joint>
@@ -159,22 +176,15 @@
      <origin xyz="0 0 0.0" rpy="0 0 0" />
      <geometry>
-       <mesh filename="package://mecanum_model/meshes/wheel_shaft_max.stl" scale="0.001 0.001 0.001"/>
+       <mesh filename="$(find mecanum_model)/meshes/wheel_shaft_max.stl" scale="0.001 0.001 0.001"/>
      </geometry>
      <material name="black" />
    </visual>
    <collision>
-     <origin xyz="0 0 0.0"/>
-     <geometry>
-       <mesh filename="package://mecanum_model/meshes/wheel_shaft_max.stl" scale="0.001 0.001 0.001"/>
-     </geometry>
-   </collision>
-   <inertial>
-     <origin xyz="0 0 0" rpy="0 0 0"/>
-     <mass value="0.055"/>
-     <inertia
-       ixx="0.000021370" ixy="0" ixz="0"
-       iyy="0.000009966" iyz="0"
-       izz="0.000021370"/>
-   </inertial>
+      <origin rpy="0 0 0" xyz="0 0 0"/>
+      <geometry>
+        <box size="${32.400002 * 0.001} ${37.585724 * 0.001} ${37.599998 * 0.001}"/>
+      </geometry>
+    </collision>
+    <xacro:box_inertia m="1.0" w="${32.400002 * 0.001}" d="${37.585724 * 0.001}" h="${37.599998 * 0.001}"/>
  </link>
  <joint name="wheel3_wheel_joint" type="fixed">
@@ -187,28 +197,20 @@
       <origin xyz="0 0 0" rpy="0 0 0"/>
       <geometry>
-      	<mesh filename="package://mecanum_model/meshes/wheel_cw.stl" scale="0.001 0.001 0.001"/>
-	     </geometry>
-       <material name="light_grey" />
-    </visual>
-    <collision>
-      <origin xyz="0 0 0" rpy="0 0 0"/>
-      <geometry>
-        <cylinder radius="${wheel_radius}" length="${wheel_width}"/>
-      </geometry>
-    </collision>
-    <inertial>
-      <origin xyz="0 0 0.0" rpy="0 0 0"/>
-      <mass value="0.3844"/>
-      <!-- Inertia based on cylinder -->
-      <inertia
-        ixx="0.000324824" ixy="0" ixz="0"
-        iyy="0.000480000" iyz="0"
-        izz="0.000324824"/>
-    </inertial>
+      	<mesh filename="$(find mecanum_model)/meshes/wheel_cw.stl" scale="0.001 0.001 0.001"/>
+	     </geometry>
+       <material name="light_grey" />
+    </visual>
+    <collision>
+      <origin rpy="0 0 0" xyz="0 0 0"/>
+      <geometry>
+        <box size="${45.538025  * 0.001} ${102.041016 * 0.001} ${102.040993 * 0.001}"/>
+      </geometry>
+    </collision>
+    <xacro:box_inertia m="1.0" w="${45.538025 * 0.001}" d="${102.041016 * 0.001}" h="${102.040993 * 0.001}"/>
   </link>
    <joint name="wheel4_shaft_joint" type="continuous">
      <origin xyz="-0.065 -0.1 0.0" rpy="0 0 0" />
       <axis xyz="1 0 0"/>
-     <parent link="base_link"/>
+     <parent link="chassis"/>
      <child link="wheel4_shaft" />
   </joint>
@@ -217,22 +219,15 @@
      <origin xyz="0 0 0.0" rpy="0 0 0" />
      <geometry>
-       <mesh filename="package://mecanum_model/meshes/wheel_shaft_min.stl" scale="0.001 0.001 0.001"/>
+       <mesh filename="$(find mecanum_model)/meshes/wheel_shaft_min.stl" scale="0.001 0.001 0.001"/>
      </geometry>
      <material name="black" />
    </visual>
    <collision>
-     <origin xyz="0 0 0.0"/>
-     <geometry>
-       <mesh filename="package://mecanum_model/meshes/wheel_shaft_min.stl" scale="0.001 0.001 0.001"/>
-     </geometry>
-   </collision>
-   <inertial>
-     <origin xyz="0 0 0" rpy="0 0 0"/>
-     <mass value="0.055"/>
-     <inertia
-       ixx="0.000021370" ixy="0" ixz="0"
-       iyy="0.000009966" iyz="0"
-       izz="0.000021370"/>
-   </inertial>
+      <origin rpy="0 0 0" xyz="0 0 0"/>
+      <geometry>
+        <box size="${32.400002 * 0.001} ${37.585724 * 0.001} ${37.599998 * 0.001}"/>
+      </geometry>
+    </collision>
+    <xacro:box_inertia m="1.0" w="${32.400002 * 0.001}" d="${37.585724 * 0.001}" h="${37.599998 * 0.001}"/>
  </link>
  <joint name="wheel4_wheel_joint" type="fixed">
@@ -245,23 +240,15 @@
       <origin xyz="0 0 0" rpy="0 0 0"/>
       <geometry>
-      	<mesh filename="package://mecanum_model/meshes/wheel_ccw.stl" scale="0.001 0.001 0.001"/>
-	     </geometry>
-       <material name="light_grey" />
-    </visual>
-    <collision>
-      <origin xyz="0 0 0" rpy="0 0 0"/>
-      <geometry>
-        <cylinder radius="${wheel_radius}" length="${wheel_width}"/>
-      </geometry>
-    </collision>
-    <inertial>
-      <origin xyz="0 0 0.0" rpy="0 0 0"/>
-      <mass value="0.3844"/>
-      <!-- Inertia based on cylinder -->
-      <inertia
-        ixx="0.000324824" ixy="0" ixz="0"
-        iyy="0.000480000" iyz="0"
-        izz="0.000324824"/>
-    </inertial>
+      	<mesh filename="$(find mecanum_model)/meshes/wheel_ccw.stl" scale="0.001 0.001 0.001"/>
+	     </geometry>
+       <material name="light_grey" />
+    </visual>
+    <collision>
+      <origin rpy="0 0 0" xyz="0 0 0"/>
+      <geometry>
+        <box size="${45.538025  * 0.001} ${102.041016 * 0.001} ${102.040993 * 0.001}"/>
+      </geometry>
+    </collision>
+    <xacro:box_inertia m="1.0" w="${45.538025 * 0.001}" d="${102.041016 * 0.001}" h="${102.040993 * 0.001}"/>
   </link>
 </robot>
