Commit message: fix mesh references

File: src/mecanum_model/urdf/s1-based-rover.urdf.xacro (robot description, xacro)
@@ -2,6 +2,6 @@
 <robot name="rover" xmlns:xacro="http://ros.org/wiki/xacro">
   <xacro:property name="PI" value="3.1415926535897931" />
-  <xacro:property name="wheel_radius" value="0.050" />
-  <xacro:property name="wheel_width" value="0.0505" />
+  <xacro:property name="wheel_radius" value="${102.041016 / 2 * 0.001}" />
+  <xacro:property name="wheel_width" value="${45.538025 * 0.001}" />
   <material name="black"><color rgba="0.15 0.15 0.15 1.0" /></material>
   <material name="light_grey"><color rgba="0.4 0.4 0.4 1.0" /></material>
@@ -48,5 +48,5 @@
     <visual>
       <geometry>
-        <mesh filename="$(find mecanum_model)/meshes/chassis.stl" scale="0.001 0.001 0.001"/>
+        <mesh filename="file://$(find mecanum_model)/meshes/chassis.stl" scale="0.001 0.001 0.001"/>
        </geometry>
        <material name="black" />
@@ -68,5 +68,5 @@
     <visual>
       <geometry>
-        <mesh filename="$(find mecanum_model)/meshes/sprayer_assembly.stl" scale="0.001 0.001 0.001"/>
+        <mesh filename="file://$(find mecanum_model)/meshes/sprayer_assembly.stl" scale="0.001 0.001 0.001"/>
        </geometry>
        <material name="light_grey" />
@@ -90,5 +90,5 @@
      <origin xyz="0 0 0.0" rpy="0 0 0" />
      <geometry>
-       <mesh filename="$(find mecanum_model)/meshes/wheel_shaft_min.stl" scale="0.001 0.001 0.001"/>
+       <mesh filename="file://$(find mecanum_model)/meshes/wheel_shaft_min.stl" scale="0.001 0.001 0.001"/>
      </geometry>
      <material name="black" />
@@ -111,21 +111,21 @@
       <origin xyz="0 0 0" rpy="0 0 0"/>
       <geometry>
-      	<mesh filename="$(find mecanum_model)/meshes/wheel_cw.stl" scale="0.001 0.001 0.001"/>
-	     </geometry>
-       <material name="light_grey" />
-    </visual>
-     <collision>
-      <origin rpy="0 0 0" xyz="0 0 0"/>
-      <geometry>
-        <box size="${10  * 0.001} ${10* 0.001} ${102.040993 * 0.001}"/>
-      </geometry>
-    </collision>
-    <xacro:box_inertia m="1.0" w="${45.538025 * 0.001}" d="${102.041016 * 0.001}" h="${102.040993 * 0.001}"/>
-  </link>
-    <joint name="wheel2_shaft_joint" type="continuous">
-     <origin xyz="0.065 0.1 0.0" rpy="0 0 0" />
-      <axis xyz="1 0 0"/>
-     <parent link="chassis"/>
-     <child link="wheel2_shaft" />
+      	<mesh filename="file://$(find mecanum_model)/meshes/wheel_cw.stl" scale="0.001 0.001 0.001"/>
+	     </geometry>
+       <material name="light_grey" />
+    </visual>
+    <collision>
+      <origin rpy="${PI/2} 0 0" xyz="0 0 0"/>
+      <geometry>
+        <cylinder length="${wheel_width}" radius="${wheel_radius}" />
+      </geometry>
+    </collision>
+    <xacro:cylinder_inertia m="1.0" r="${wheel_radius}" h="${wheel_width}"/>
+  </link>
+  <joint name="wheel2_shaft_joint" type="continuous">
+    <origin xyz="0.065 0.1 0.0" rpy="0 0 0" />
+    <axis xyz="1 0 0"/>
+    <parent link="chassis"/>
+    <child link="wheel2_shaft" />
   </joint>
   <link name="wheel2_shaft">
@@ -133,5 +133,5 @@
      <origin xyz="0 0 0.0" rpy="0 0 0" />
      <geometry>
-       <mesh filename="$(find mecanum_model)/meshes/wheel_shaft_max.stl" scale="0.001 0.001 0.001"/>
+       <mesh filename="file://$(find mecanum_model)/meshes/wheel_shaft_max.stl" scale="0.001 0.001 0.001"/>
      </geometry>
      <material name="black" />
@@ -154,15 +154,15 @@
       <origin xyz="0 0 0" rpy="0 0 0"/>
       <geometry>
-      	<mesh filename="$(find mecanum_model)/meshes/wheel_ccw.stl" scale="0.001 0.001 0.001"/>
-	     </geometry>
-       <material name="light_grey" />
-    </visual>
-    <collision>
-      <origin rpy="0 0 0" xyz="0 0 0"/>
-      <geometry>
-        <box size="${45.538025  * 0.001} ${102.041016 * 0.001} ${102.040993 * 0.001}"/>
-      </geometry>
-    </collision>
-    <xacro:box_inertia m="1.0" w="${45.538025 * 0.001}" d="${102.041016 * 0.001}" h="${102.040993 * 0.001}"/>
+      	<mesh filename="file://$(find mecanum_model)/meshes/wheel_ccw.stl" scale="0.001 0.001 0.001"/>
+	     </geometry>
+       <material name="light_grey" />
+    </visual>
+    <collision>
+      <origin rpy="${PI/2} 0 0" xyz="0 0 0"/>
+      <geometry>
+        <cylinder length="${wheel_width}" radius="${wheel_radius}" />
+      </geometry>
+    </collision>
+    <xacro:cylinder_inertia m="1.0" r="${wheel_radius}" h="${wheel_width}"/>
   </link>
    <joint name="wheel3_shaft_joint" type="continuous">
@@ -176,5 +176,5 @@
      <origin xyz="0 0 0.0" rpy="0 0 0" />
      <geometry>
-       <mesh filename="$(find mecanum_model)/meshes/wheel_shaft_max.stl" scale="0.001 0.001 0.001"/>
+       <mesh filename="file://$(find mecanum_model)/meshes/wheel_shaft_max.stl" scale="0.001 0.001 0.001"/>
      </geometry>
      <material name="black" />
@@ -197,15 +197,15 @@
       <origin xyz="0 0 0" rpy="0 0 0"/>
       <geometry>
-      	<mesh filename="$(find mecanum_model)/meshes/wheel_cw.stl" scale="0.001 0.001 0.001"/>
-	     </geometry>
-       <material name="light_grey" />
-    </visual>
-    <collision>
-      <origin rpy="0 0 0" xyz="0 0 0"/>
-      <geometry>
-        <box size="${45.538025  * 0.001} ${102.041016 * 0.001} ${102.040993 * 0.001}"/>
-      </geometry>
-    </collision>
-    <xacro:box_inertia m="1.0" w="${45.538025 * 0.001}" d="${102.041016 * 0.001}" h="${102.040993 * 0.001}"/>
+      	<mesh filename="file://$(find mecanum_model)/meshes/wheel_cw.stl" scale="0.001 0.001 0.001"/>
+	     </geometry>
+       <material name="light_grey" />
+    </visual>
+    <collision>
+      <origin rpy="${PI/2} 0 0" xyz="0 0 0"/>
+      <geometry>
+        <cylinder length="${wheel_width}" radius="${wheel_radius}" />
+      </geometry>
+    </collision>
+    <xacro:cylinder_inertia m="1.0" r="${wheel_radius}" h="${wheel_width}"/>
   </link>
    <joint name="wheel4_shaft_joint" type="continuous">
@@ -219,5 +219,5 @@
      <origin xyz="0 0 0.0" rpy="0 0 0" />
      <geometry>
-       <mesh filename="$(find mecanum_model)/meshes/wheel_shaft_min.stl" scale="0.001 0.001 0.001"/>
+       <mesh filename="file://$(find mecanum_model)/meshes/wheel_shaft_min.stl" scale="0.001 0.001 0.001"/>
      </geometry>
      <material name="black" />
@@ -240,15 +240,15 @@
       <origin xyz="0 0 0" rpy="0 0 0"/>
       <geometry>
-      	<mesh filename="$(find mecanum_model)/meshes/wheel_ccw.stl" scale="0.001 0.001 0.001"/>
-	     </geometry>
-       <material name="light_grey" />
-    </visual>
-    <collision>
-      <origin rpy="0 0 0" xyz="0 0 0"/>
-      <geometry>
-        <box size="${45.538025  * 0.001} ${102.041016 * 0.001} ${102.040993 * 0.001}"/>
-      </geometry>
-    </collision>
-    <xacro:box_inertia m="1.0" w="${45.538025 * 0.001}" d="${102.041016 * 0.001}" h="${102.040993 * 0.001}"/>
+      	<mesh filename="file://$(find mecanum_model)/meshes/wheel_ccw.stl" scale="0.001 0.001 0.001"/>
+	     </geometry>
+       <material name="light_grey" />
+    </visual>
+    <collision>
+      <origin rpy="${PI/2} 0 0" xyz="0 0 0"/>
+      <geometry>
+        <cylinder length="${wheel_width}" radius="${wheel_radius}" />
+      </geometry>
+    </collision>
+    <xacro:cylinder_inertia m="1.0" r="${wheel_radius}" h="${wheel_width}"/>
   </link>
 </robot>

Commit message: fix wheel orientation and collisions

File: src/mecanum_model/urdf/s1-based-rover.urdf.xacro (robot description, xacro)
@@ -4,4 +4,6 @@
   <xacro:property name="wheel_radius" value="${102.041016 / 2 * 0.001}" />
   <xacro:property name="wheel_width" value="${45.538025 * 0.001}" />
+  <xacro:property name="wheel_shaft_radius" value="${5.0 * 0.001}" />
+  <xacro:property name="wheel_shaft_length" value="${37.585724 * 0.001}" />
   <material name="black"><color rgba="0.15 0.15 0.15 1.0" /></material>
   <material name="light_grey"><color rgba="0.4 0.4 0.4 1.0" /></material>
@@ -94,11 +96,11 @@
      <material name="black" />
    </visual>
-   <collision>
-      <origin rpy="0 0 0" xyz="0 0 0"/>
-      <geometry>
-        <box size="${32.400002 * 0.001} ${37.585724 * 0.001} ${37.599998 * 0.001}"/>
-      </geometry>
-    </collision>
-    <xacro:box_inertia m="1.0" w="${32.400002 * 0.001}" d="${37.585724 * 0.001}" h="${37.599998 * 0.001}"/>
+    <collision>
+      <origin rpy="${PI/2} 0 0" xyz="0 0 0"/>
+      <geometry>
+        <cylinder length="${wheel_shaft_length}" radius="${wheel_shaft_radius}" />
+      </geometry>
+    </collision>
+    <xacro:cylinder_inertia m="1.0" r="${wheel_shaft_radius}" h="${wheel_shaft_length}"/>
  </link>
  <joint name="wheel1_wheel_joint" type="fixed">
@@ -138,10 +140,10 @@
    </visual>
     <collision>
-      <origin rpy="0 0 0" xyz="0 0 0"/>
-      <geometry>
-        <box size="${32.400002 * 0.001} ${37.585724 * 0.001} ${37.599998 * 0.001}"/>
-      </geometry>
-    </collision>
-    <xacro:box_inertia m="1.0" w="${32.400002 * 0.001}" d="${37.585724 * 0.001}" h="${37.599998 * 0.001}"/>
+      <origin rpy="${PI/2} 0 0" xyz="0 0 0"/>
+      <geometry>
+        <cylinder length="${wheel_shaft_length}" radius="${wheel_shaft_radius}" />
+      </geometry>
+    </collision>
+    <xacro:cylinder_inertia m="1.0" r="${wheel_shaft_radius}" h="${wheel_shaft_length}"/>
  </link>
  <joint name="wheel2_wheel_joint" type="fixed">
@@ -181,10 +183,10 @@
    </visual>
    <collision>
-      <origin rpy="0 0 0" xyz="0 0 0"/>
-      <geometry>
-        <box size="${32.400002 * 0.001} ${37.585724 * 0.001} ${37.599998 * 0.001}"/>
-      </geometry>
-    </collision>
-    <xacro:box_inertia m="1.0" w="${32.400002 * 0.001}" d="${37.585724 * 0.001}" h="${37.599998 * 0.001}"/>
+      <origin rpy="${PI/2} 0 0" xyz="0 0 0"/>
+      <geometry>
+        <cylinder length="${wheel_shaft_length}" radius="${wheel_shaft_radius}" />
+      </geometry>
+    </collision>
+    <xacro:cylinder_inertia m="1.0" r="${wheel_shaft_radius}" h="${wheel_shaft_length}"/>
  </link>
  <joint name="wheel3_wheel_joint" type="fixed">
@@ -195,5 +197,5 @@
   <link name="wheel3">
     <visual>
-      <origin xyz="0 0 0" rpy="0 0 0"/>
+      <origin xyz="0 0 0" rpy="0 0 ${PI}"/>
       <geometry>
       	<mesh filename="file://$(find mecanum_model)/meshes/wheel_cw.stl" scale="0.001 0.001 0.001"/>
@@ -223,11 +225,11 @@
      <material name="black" />
    </visual>
-   <collision>
-      <origin rpy="0 0 0" xyz="0 0 0"/>
-      <geometry>
-        <box size="${32.400002 * 0.001} ${37.585724 * 0.001} ${37.599998 * 0.001}"/>
-      </geometry>
-    </collision>
-    <xacro:box_inertia m="1.0" w="${32.400002 * 0.001}" d="${37.585724 * 0.001}" h="${37.599998 * 0.001}"/>
+    <collision>
+      <origin rpy="${PI/2} 0 0" xyz="0 0 0"/>
+      <geometry>
+        <cylinder length="${wheel_shaft_length}" radius="${wheel_shaft_radius}" />
+      </geometry>
+    </collision>
+    <xacro:cylinder_inertia m="1.0" r="${wheel_shaft_radius}" h="${wheel_shaft_length}"/>
  </link>
  <joint name="wheel4_wheel_joint" type="fixed">
@@ -238,5 +240,5 @@
   <link name="wheel4">
     <visual>
-      <origin xyz="0 0 0" rpy="0 0 0"/>
+      <origin xyz="0 0 0" rpy="0 0 ${PI}"/>
       <geometry>
       	<mesh filename="file://$(find mecanum_model)/meshes/wheel_ccw.stl" scale="0.001 0.001 0.001"/>
