Commit message: new parametric wheels

File: src/mecanum_model/urdf/s1-based-rover.urdf (robot description, URDF)
Before this commit: robot rover, 12 links, 11 joints
Links:
- removed link wheel1
- added link front_left_roller10_link, mass 0.3; collision mesh filename=file:///home/johnathan/devel/inspectobot/rosrover/install/m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 scale=1 1 1; visual mesh filename=file:///home/johnathan/devel/inspectobot/rosrover/install/m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 scale=0.001 0.001 0.001
- added link front_left_roller11_link, mass 0.3; collision mesh filename=file:///home/johnathan/devel/inspectobot/rosrover/install/m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 scale=1 1 1; visual mesh filename=file:///home/johnathan/devel/inspectobot/rosrover/install/m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 scale=0.001 0.001 0.001
- added link front_left_roller12_link, mass 0.3; collision mesh filename=file:///home/johnathan/devel/inspectobot/rosrover/install/m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 scale=1 1 1; visual mesh filename=file:///home/johnathan/devel/inspectobot/rosrover/install/m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 scale=0.001 0.001 0.001
- added link front_left_roller13_link, mass 0.3; collision mesh filename=file:///home/johnathan/devel/inspectobot/rosrover/install/m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 scale=1 1 1; visual mesh filename=file:///home/johnathan/devel/inspectobot/rosrover/install/m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 scale=0.001 0.001 0.001
- added link front_left_roller14_link, mass 0.3; collision mesh filename=file:///home/johnathan/devel/inspectobot/rosrover/install/m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 scale=1 1 1; visual mesh filename=file:///home/johnathan/devel/inspectobot/rosrover/install/m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 scale=0.001 0.001 0.001
- added link front_left_roller15_link, mass 0.3; collision mesh filename=file:///home/johnathan/devel/inspectobot/rosrover/install/m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 scale=1 1 1; visual mesh filename=file:///home/johnathan/devel/inspectobot/rosrover/install/m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 scale=0.001 0.001 0.001
- added link front_left_roller1_link, mass 0.3; collision mesh filename=file:///home/johnathan/devel/inspectobot/rosrover/install/m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 scale=1 1 1; visual mesh filename=file:///home/johnathan/devel/inspectobot/rosrover/install/m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 scale=0.001 0.001 0.001
- added link front_left_roller2_link, mass 0.3; collision mesh filename=file:///home/johnathan/devel/inspectobot/rosrover/install/m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 scale=1 1 1; visual mesh filename=file:///home/johnathan/devel/inspectobot/rosrover/install/m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 scale=0.001 0.001 0.001
- added link front_left_roller3_link, mass 0.3; collision mesh filename=file:///home/johnathan/devel/inspectobot/rosrover/install/m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 scale=1 1 1; visual mesh filename=file:///home/johnathan/devel/inspectobot/rosrover/install/m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 scale=0.001 0.001 0.001
- added link front_left_roller4_link, mass 0.3; collision mesh filename=file:///home/johnathan/devel/inspectobot/rosrover/install/m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 scale=1 1 1; visual mesh filename=file:///home/johnathan/devel/inspectobot/rosrover/install/m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 scale=0.001 0.001 0.001
- added link front_left_roller5_link, mass 0.3; collision mesh filename=file:///home/johnathan/devel/inspectobot/rosrover/install/m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 scale=1 1 1; visual mesh filename=file:///home/johnathan/devel/inspectobot/rosrover/install/m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 scale=0.001 0.001 0.001
- added link front_left_roller6_link, mass 0.3; collision mesh filename=file:///home/johnathan/devel/inspectobot/rosrover/install/m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 scale=1 1 1; visual mesh filename=file:///home/johnathan/devel/inspectobot/rosrover/install/m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 scale=0.001 0.001 0.001
- added link front_left_roller7_link, mass 0.3; collision mesh filename=file:///home/johnathan/devel/inspectobot/rosrover/install/m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 scale=1 1 1; visual mesh filename=file:///home/johnathan/devel/inspectobot/rosrover/install/m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 scale=0.001 0.001 0.001
- added link front_left_roller8_link, mass 0.3; collision mesh filename=file:///home/johnathan/devel/inspectobot/rosrover/install/m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 scale=1 1 1; visual mesh filename=file:///home/johnathan/devel/inspectobot/rosrover/install/m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 scale=0.001 0.001 0.001
- added link front_left_roller9_link, mass 0.3; collision mesh filename=file:///home/johnathan/devel/inspectobot/rosrover/install/m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 scale=1 1 1; visual mesh filename=file:///home/johnathan/devel/inspectobot/rosrover/install/m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 scale=0.001 0.001 0.001
- added link front_left_wheel_link, mass 2.0; collision mesh filename=file:///home/johnathan/devel/inspectobot/rosrover/install/m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 scale=-0.001 0.001 0.001; visual mesh filename=file:///home/johnathan/devel/inspectobot/rosrover/install/m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 scale=-0.001 0.001 0.001
- link base_footprint: mass 1 -> None; geometry collision box size=0.24486561599999998 0.302041534 0.102041229
- link chassis: mass 1 -> 1.0; geometry collision box size=0.14839953600000003 0.252206665 0.055450001; visual mesh filename=file:///home/johnathan/devel/inspectobot/rosrover/install/m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 scale=0.001 0.001 0.001
- link sprayer_assembly: mass None -> 1.0; geometry collision box size=0.144179398 0.069498428 0.096728165; visual mesh filename=file:///home/johnathan/devel/inspectobot/rosrover/install/m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 scale=0.001 0.001 0.001
- link wheel1_shaft: mass 0.055 -> 1.0; geometry collision cylinder length=0.037585724 radius=0.005; visual mesh filename=file:///home/johnathan/devel/inspectobot/rosrover/install/m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 scale=0.001 0.001 0.001
- link wheel2: mass 0.3844 -> 1.0; geometry collision cylinder length=0.045538024999999996 radius=0.051020508; visual mesh filename=file:///home/johnathan/devel/inspectobot/rosrover/install/m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 scale=0.001 0.001 0.001
- link wheel2_shaft: mass 0.055 -> 1.0; geometry collision cylinder length=0.037585724 radius=0.005; visual mesh filename=file:///home/johnathan/devel/inspectobot/rosrover/install/m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 scale=0.001 0.001 0.001
- link wheel3: mass 0.3844 -> 1.0; geometry collision cylinder length=0.045538024999999996 radius=0.051020508; visual mesh filename=file:///home/johnathan/devel/inspectobot/rosrover/install/m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 scale=0.001 0.001 0.001
- link wheel3_shaft: mass 0.055 -> 1.0; geometry collision cylinder length=0.037585724 radius=0.005; visual mesh filename=file:///home/johnathan/devel/inspectobot/rosrover/install/m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 scale=0.001 0.001 0.001
- link wheel4: mass 0.3844 -> 1.0; geometry collision cylinder length=0.045538024999999996 radius=0.051020508; visual mesh filename=file:///home/johnathan/devel/inspectobot/rosrover/install/m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 scale=0.001 0.001 0.001
- link wheel4_shaft: mass 0.055 -> 1.0; geometry collision cylinder length=0.037585724 radius=0.005; visual mesh filename=file:///home/johnathan/devel/inspectobot/rosrover/install/m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 scale=0.001 0.001 0.001
Joints:
- added joint front_left_roller10_joint: type continuous, parent front_left_wheel_link, child front_left_roller10_link, origin xyz=0 -0.0362035104982789 -0.02630339004008817 rpy=-0.7989541677433551 0.6090169187607924 0.5313896516603533
- added joint front_left_roller11_joint: type continuous, parent front_left_wheel_link, child front_left_roller11_link, origin xyz=0 -0.02237500000000002 -0.038754636819353615 rpy=-1.1831996401397156 0.3613671239067081 0.7137243789447655
- added joint front_left_roller12_joint: type continuous, parent front_left_wheel_link, child front_left_roller12_link, origin xyz=0 -0.004677648731227488 -0.044504854817730234 rpy=-1.4966127917301506 0.07398025001120935 0.7826515949744619
- added joint front_left_roller13_joint: type continuous, parent front_left_wheel_link, child front_left_roller13_link, origin xyz=0 0.013828510498278887 -0.04255977910420812 rpy=1.3449626171032882 -0.22028527385474703 0.7603177925108144
- added joint front_left_roller14_joint: type continuous, parent front_left_wheel_link, child front_left_roller14_link, origin xyz=0 0.029943594634558885 -0.03325573094011341 rpy=1.0038406803226874 -0.4928592704898482 0.6390993414905143
- added joint front_left_roller15_joint: type continuous, parent front_left_wheel_link, child front_left_roller15_link, origin xyz=0 0.04088115922950639 -0.018201464777642055 rpy=0.5619350361043127 -0.7022987807291682 0.38630030387691144
- added joint front_left_roller1_joint: type continuous, parent front_left_wheel_link, child front_left_roller1_link, origin xyz=0 0.04475 0.0 rpy=-0.0 -0.7853981633974482 -0.0
- added joint front_left_roller2_joint: type continuous, parent front_left_wheel_link, child front_left_roller2_link, origin xyz=0 0.040881159229506386 0.01820146477764206 rpy=-0.5619350361043128 -0.702298780729168 -0.3863003038769115
- added joint front_left_roller3_joint: type continuous, parent front_left_wheel_link, child front_left_roller3_link, origin xyz=0 0.029943594634558906 0.033255730940113394 rpy=-1.0038406803226867 -0.4928592704898485 -0.6390993414905141
- added joint front_left_roller4_joint: type continuous, parent front_left_wheel_link, child front_left_roller4_link, origin xyz=0 0.013828510498278898 0.04255977910420812 rpy=-1.3449626171032882 -0.2202852738547472 -0.7603177925108144
- added joint front_left_roller5_joint: type continuous, parent front_left_wheel_link, child front_left_roller5_link, origin xyz=0 -0.0046776487312274965 0.04450485481773023 rpy=1.4966127917301504 0.07398025001120949 -0.7826515949744619
- added joint front_left_roller6_joint: type continuous, parent front_left_wheel_link, child front_left_roller6_link, origin xyz=0 -0.02237499999999999 0.03875463681935363 rpy=1.1831996401397162 0.3613671239067076 -0.7137243789447657
- added joint front_left_roller7_joint: type continuous, parent front_left_wheel_link, child front_left_roller7_link, origin xyz=0 -0.03620351049827889 0.026303390040088175 rpy=0.7989541677433554 0.6090169187607923 -0.5313896516603536
- added joint front_left_roller8_joint: type continuous, parent front_left_wheel_link, child front_left_roller8_link, origin xyz=0 -0.0437721051328378 0.00930404816409473 rpy=0.2920075036845471 0.7637777909460687 -0.20499125187874387
- added joint front_left_roller9_joint: type continuous, parent front_left_wheel_link, child front_left_roller9_link, origin xyz=0 -0.043772105132837795 -0.009304048164094738 rpy=-0.29200750368454736 0.7637777909460687 0.20499125187874406
- joint wheel1_wheel_joint: child wheel1 -> front_left_wheel_link

File: src/mecanum_model/urdf/s1-based-rover.urdf.xacro (robot description, xacro)
@@ -29,4 +29,5 @@
   </xacro:macro>
   <xacro:include filename="$(find mecanum_model)/urdf/s1-based-rover.gazebo" />
+  <xacro:include filename="$(find mecanum_model)/urdf/mecanum/mecanum_wheel_macro.xacro" />
   <link name="world"></link>
   <joint name="fixed" type="fixed">
@@ -50,5 +51,5 @@
     <visual>
       <geometry>
-        <mesh filename="file://$(find mecanum_model)/meshes/chassis.stl" scale="0.001 0.001 0.001"/>
+        <mesh filename="file://$(find mecanum_model)/meshes/visual/chassis.stl" scale="0.001 0.001 0.001"/>
        </geometry>
        <material name="black" />
@@ -70,5 +71,5 @@
     <visual>
       <geometry>
-        <mesh filename="file://$(find mecanum_model)/meshes/sprayer_assembly.stl" scale="0.001 0.001 0.001"/>
+        <mesh filename="file://$(find mecanum_model)/meshes/visual/sprayer_assembly.stl" scale="0.001 0.001 0.001"/>
        </geometry>
        <material name="light_grey" />
@@ -92,5 +93,5 @@
      <origin xyz="0 0 0.0" rpy="0 0 0" />
      <geometry>
-       <mesh filename="file://$(find mecanum_model)/meshes/wheel_shaft_min.stl" scale="0.001 0.001 0.001"/>
+       <mesh filename="file://$(find mecanum_model)/meshes/visual/wheel_shaft_min.stl" scale="0.001 0.001 0.001"/>
      </geometry>
      <material name="black" />
@@ -107,22 +108,7 @@
    <origin xyz="-0.035 0 0" rpy="0 0 0" />
    <parent link="wheel1_shaft"/>
-   <child link="wheel1" />
+   <child link="front_left_wheel_link" />
  </joint>
-  <link name="wheel1">
-    <visual>
-      <origin xyz="0 0 0" rpy="0 0 0"/>
-      <geometry>
-      	<mesh filename="file://$(find mecanum_model)/meshes/wheel_cw.stl" scale="0.001 0.001 0.001"/>
-	     </geometry>
-       <material name="light_grey" />
-    </visual>
-    <collision>
-      <origin rpy="${PI/2} 0 0" xyz="0 0 0"/>
-      <geometry>
-        <cylinder length="${wheel_width}" radius="${wheel_radius}" />
-      </geometry>
-    </collision>
-    <xacro:cylinder_inertia m="1.0" r="${wheel_radius}" h="${wheel_width}"/>
-  </link>
+  <xacro:mecanum_wheel name="front_left"  side="-1" interface="hardware_interface/EffortJointInterface"/>
   <joint name="wheel2_shaft_joint" type="continuous">
     <origin xyz="0.065 0.1 0.0" rpy="0 0 0" />
@@ -135,5 +121,5 @@
      <origin xyz="0 0 0.0" rpy="0 0 0" />
      <geometry>
-       <mesh filename="file://$(find mecanum_model)/meshes/wheel_shaft_max.stl" scale="0.001 0.001 0.001"/>
+       <mesh filename="file://$(find mecanum_model)/meshes/visual/wheel_shaft_max.stl" scale="0.001 0.001 0.001"/>
      </geometry>
      <material name="black" />
@@ -150,22 +136,7 @@
    <origin xyz="0.035 0 0" rpy="0 0 0" />
    <parent link="wheel2_shaft"/>
-   <child link="wheel2" />
+   <child link="front_right_wheel_link" />
  </joint>
-  <link name="wheel2">
-    <visual>
-      <origin xyz="0 0 0" rpy="0 0 0"/>
-      <geometry>
-      	<mesh filename="file://$(find mecanum_model)/meshes/wheel_ccw.stl" scale="0.001 0.001 0.001"/>
-	     </geometry>
-       <material name="light_grey" />
-    </visual>
-    <collision>
-      <origin rpy="${PI/2} 0 0" xyz="0 0 0"/>
-      <geometry>
-        <cylinder length="${wheel_width}" radius="${wheel_radius}" />
-      </geometry>
-    </collision>
-    <xacro:cylinder_inertia m="1.0" r="${wheel_radius}" h="${wheel_width}"/>
-  </link>
+ <xacro:mecanum_wheel name="front_right"  side="1" interface="hardware_interface/EffortJointInterface"/>
    <joint name="wheel3_shaft_joint" type="continuous">
      <origin xyz="0.065 -0.1 0.0" rpy="0 0 0" />
@@ -178,5 +149,5 @@
      <origin xyz="0 0 0.0" rpy="0 0 0" />
      <geometry>
-       <mesh filename="file://$(find mecanum_model)/meshes/wheel_shaft_max.stl" scale="0.001 0.001 0.001"/>
+       <mesh filename="file://$(find mecanum_model)/meshes/visual/wheel_shaft_max.stl" scale="0.001 0.001 0.001"/>
      </geometry>
      <material name="black" />
@@ -193,22 +164,7 @@
    <origin xyz="0.035 0 0" rpy="0 0 0" />
    <parent link="wheel3_shaft"/>
-   <child link="wheel3" />
+   <child link="rear_right_wheel_link" />
  </joint>
-  <link name="wheel3">
-    <visual>
-      <origin xyz="0 0 0" rpy="0 0 ${PI}"/>
-      <geometry>
-      	<mesh filename="file://$(find mecanum_model)/meshes/wheel_cw.stl" scale="0.001 0.001 0.001"/>
-	     </geometry>
-       <material name="light_grey" />
-    </visual>
-    <collision>
-      <origin rpy="${PI/2} 0 0" xyz="0 0 0"/>
-      <geometry>
-        <cylinder length="${wheel_width}" radius="${wheel_radius}" />
-      </geometry>
-    </collision>
-    <xacro:cylinder_inertia m="1.0" r="${wheel_radius}" h="${wheel_width}"/>
-  </link>
+  <xacro:mecanum_wheel name="rear_right"  side="1" interface="hardware_interface/EffortJointInterface"/>
    <joint name="wheel4_shaft_joint" type="continuous">
      <origin xyz="-0.065 -0.1 0.0" rpy="0 0 0" />
@@ -221,5 +177,5 @@
      <origin xyz="0 0 0.0" rpy="0 0 0" />
      <geometry>
-       <mesh filename="file://$(find mecanum_model)/meshes/wheel_shaft_min.stl" scale="0.001 0.001 0.001"/>
+       <mesh filename="file://$(find mecanum_model)/meshes/visual/wheel_shaft_min.stl" scale="0.001 0.001 0.001"/>
      </geometry>
      <material name="black" />
@@ -236,21 +192,6 @@
    <origin xyz="-0.035 0 0" rpy="0 0 0" />
    <parent link="wheel4_shaft"/>
-   <child link="wheel4" />
+   <child link="rear_left_wheel_link" />
  </joint>
-  <link name="wheel4">
-    <visual>
-      <origin xyz="0 0 0" rpy="0 0 ${PI}"/>
-      <geometry>
-      	<mesh filename="file://$(find mecanum_model)/meshes/wheel_ccw.stl" scale="0.001 0.001 0.001"/>
-	     </geometry>
-       <material name="light_grey" />
-    </visual>
-    <collision>
-      <origin rpy="${PI/2} 0 0" xyz="0 0 0"/>
-      <geometry>
-        <cylinder length="${wheel_width}" radius="${wheel_radius}" />
-      </geometry>
-    </collision>
-    <xacro:cylinder_inertia m="1.0" r="${wheel_radius}" h="${wheel_width}"/>
-  </link>
+   <xacro:mecanum_wheel name="rear_left"  side="-1" interface="hardware_interface/EffortJointInterface"/>
 </robot>
