Commit message: fixup rover model

File: src/mecanum_model/urdf/mecanum/rollers.xacro (robot description, xacro)
@@ -21,10 +21,10 @@
         <collision>
           <geometry>
-            <mesh filename="file://$(find mecanum_model)/meshes/collision/roller.stl" scale="1 1 1" />
+            <mesh filename="file://$(find mecanum_model)/meshes/collision/roller.stl" scale="0.001 0.001 0.001" />
           </geometry>
         </collision>
         <inertial>
           <origin xyz="0 0 0" />
-          <mass value="0.3" />
+          <mass value="0.15" />
           <inertia ixx="0.00024000" ixy="0.0" ixz="0.0"
                   iyy="0.00076000" iyz="0.0"
@@ -52,5 +52,5 @@
         <mu2 value="0.8"/>
         <kp value="10000000.0" />
-        <kd value="1.0" />
+        <kd value="100.0" />
         <fdir1 value="0 1 0"/>
       </gazebo>

File: src/mecanum_model/urdf/mecanum/wheel.xacro (robot description, xacro)
@@ -16,5 +16,5 @@
       <inertial>
         <origin xyz="0 0 0" />
-        <mass value="2.0" />
+        <mass value="1.0" />
         <inertia ixx="0.042025" ixy="0.0" ixz="0.0"
                 iyy="0.024279" iyz="0.0"
