Commit message: fixup rover model

File: src/mecanum_model/urdf/s1-based-rover.urdf (robot description, URDF)
Before this commit: robot rover, 27 links, 26 joints
Links:
- removed link wheel2
- removed link wheel3
- removed link wheel4
- added link front_right_roller10_link, mass 0.15; collision mesh filename=file:///home/johnathan/devel/inspectobot/rosrover/install/m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 scale=1 1 1; visual mesh filename=file:///home/johnathan/devel/inspectobot/rosrover/install/m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 scale=0.001 0.001 0.001
- added link front_right_roller11_link, mass 0.15; collision mesh filename=file:///home/johnathan/devel/inspectobot/rosrover/install/m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 scale=1 1 1; visual mesh filename=file:///home/johnathan/devel/inspectobot/rosrover/install/m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 scale=0.001 0.001 0.001
- added link front_right_roller12_link, mass 0.15; collision mesh filename=file:///home/johnathan/devel/inspectobot/rosrover/install/m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 scale=1 1 1; visual mesh filename=file:///home/johnathan/devel/inspectobot/rosrover/install/m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 scale=0.001 0.001 0.001
- added link front_right_roller13_link, mass 0.15; collision mesh filename=file:///home/johnathan/devel/inspectobot/rosrover/install/m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 scale=1 1 1; visual mesh filename=file:///home/johnathan/devel/inspectobot/rosrover/install/m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 scale=0.001 0.001 0.001
- added link front_right_roller14_link, mass 0.15; collision mesh filename=file:///home/johnathan/devel/inspectobot/rosrover/install/m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 scale=1 1 1; visual mesh filename=file:///home/johnathan/devel/inspectobot/rosrover/install/m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 scale=0.001 0.001 0.001
- added link front_right_roller15_link, mass 0.15; collision mesh filename=file:///home/johnathan/devel/inspectobot/rosrover/install/m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 scale=1 1 1; visual mesh filename=file:///home/johnathan/devel/inspectobot/rosrover/install/m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 scale=0.001 0.001 0.001
- added link front_right_roller1_link, mass 0.15; collision mesh filename=file:///home/johnathan/devel/inspectobot/rosrover/install/m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 scale=1 1 1; visual mesh filename=file:///home/johnathan/devel/inspectobot/rosrover/install/m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 scale=0.001 0.001 0.001
- added link front_right_roller2_link, mass 0.15; collision mesh filename=file:///home/johnathan/devel/inspectobot/rosrover/install/m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 scale=1 1 1; visual mesh filename=file:///home/johnathan/devel/inspectobot/rosrover/install/m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 scale=0.001 0.001 0.001
- added link front_right_roller3_link, mass 0.15; collision mesh filename=file:///home/johnathan/devel/inspectobot/rosrover/install/m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 scale=1 1 1; visual mesh filename=file:///home/johnathan/devel/inspectobot/rosrover/install/m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 scale=0.001 0.001 0.001
- added link front_right_roller4_link, mass 0.15; collision mesh filename=file:///home/johnathan/devel/inspectobot/rosrover/install/m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 scale=1 1 1; visual mesh filename=file:///home/johnathan/devel/inspectobot/rosrover/install/m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 scale=0.001 0.001 0.001
- added link front_right_roller5_link, mass 0.15; collision mesh filename=file:///home/johnathan/devel/inspectobot/rosrover/install/m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 scale=1 1 1; visual mesh filename=file:///home/johnathan/devel/inspectobot/rosrover/install/m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 scale=0.001 0.001 0.001
- added link front_right_roller6_link, mass 0.15; collision mesh filename=file:///home/johnathan/devel/inspectobot/rosrover/install/m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 scale=1 1 1; visual mesh filename=file:///home/johnathan/devel/inspectobot/rosrover/install/m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 scale=0.001 0.001 0.001
- added link front_right_roller7_link, mass 0.15; collision mesh filename=file:///home/johnathan/devel/inspectobot/rosrover/install/m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 scale=1 1 1; visual mesh filename=file:///home/johnathan/devel/inspectobot/rosrover/install/m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 scale=0.001 0.001 0.001
- added link front_right_roller8_link, mass 0.15; collision mesh filename=file:///home/johnathan/devel/inspectobot/rosrover/install/m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 scale=1 1 1; visual mesh filename=file:///home/johnathan/devel/inspectobot/rosrover/install/m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 scale=0.001 0.001 0.001
- added link front_right_roller9_link, mass 0.15; collision mesh filename=file:///home/johnathan/devel/inspectobot/rosrover/install/m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 scale=1 1 1; visual mesh filename=file:///home/johnathan/devel/inspectobot/rosrover/install/m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 scale=0.001 0.001 0.001
- added link front_right_wheel_link, mass 1.0; collision mesh filename=file:///home/johnathan/devel/inspectobot/rosrover/install/m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 scale=0.001 0.001 0.001; visual mesh filename=file:///home/johnathan/devel/inspectobot/rosrover/install/m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 scale=0.001 0.001 0.001
- added link rear_left_roller10_link, mass 0.15; collision mesh filename=file:///home/johnathan/devel/inspectobot/rosrover/install/m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 scale=1 1 1; visual mesh filename=file:///home/johnathan/devel/inspectobot/rosrover/install/m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 scale=0.001 0.001 0.001
- added link rear_left_roller11_link, mass 0.15; collision mesh filename=file:///home/johnathan/devel/inspectobot/rosrover/install/m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 scale=1 1 1; visual mesh filename=file:///home/johnathan/devel/inspectobot/rosrover/install/m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 scale=0.001 0.001 0.001
- added link rear_left_roller12_link, mass 0.15; collision mesh filename=file:///home/johnathan/devel/inspectobot/rosrover/install/m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 scale=1 1 1; visual mesh filename=file:///home/johnathan/devel/inspectobot/rosrover/install/m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 scale=0.001 0.001 0.001
- added link rear_left_roller13_link, mass 0.15; collision mesh filename=file:///home/johnathan/devel/inspectobot/rosrover/install/m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 scale=1 1 1; visual mesh filename=file:///home/johnathan/devel/inspectobot/rosrover/install/m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 scale=0.001 0.001 0.001
- added link rear_left_roller14_link, mass 0.15; collision mesh filename=file:///home/johnathan/devel/inspectobot/rosrover/install/m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 scale=1 1 1; visual mesh filename=file:///home/johnathan/devel/inspectobot/rosrover/install/m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 scale=0.001 0.001 0.001
- added link rear_left_roller15_link, mass 0.15; collision mesh filename=file:///home/johnathan/devel/inspectobot/rosrover/install/m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 scale=1 1 1; visual mesh filename=file:///home/johnathan/devel/inspectobot/rosrover/install/m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 scale=0.001 0.001 0.001
- added link rear_left_roller1_link, mass 0.15; collision mesh filename=file:///home/johnathan/devel/inspectobot/rosrover/install/m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 scale=1 1 1; visual mesh filename=file:///home/johnathan/devel/inspectobot/rosrover/install/m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 scale=0.001 0.001 0.001
- added link rear_left_roller2_link, mass 0.15; collision mesh filename=file:///home/johnathan/devel/inspectobot/rosrover/install/m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 scale=1 1 1; visual mesh filename=file:///home/johnathan/devel/inspectobot/rosrover/install/m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 scale=0.001 0.001 0.001
- added link rear_left_roller3_link, mass 0.15; collision mesh filename=file:///home/johnathan/devel/inspectobot/rosrover/install/m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 scale=1 1 1; visual mesh filename=file:///home/johnathan/devel/inspectobot/rosrover/install/m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 scale=0.001 0.001 0.001
- added link rear_left_roller4_link, mass 0.15; collision mesh filename=file:///home/johnathan/devel/inspectobot/rosrover/install/m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 scale=1 1 1; visual mesh filename=file:///home/johnathan/devel/inspectobot/rosrover/install/m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 scale=0.001 0.001 0.001
- added link rear_left_roller5_link, mass 0.15; collision mesh filename=file:///home/johnathan/devel/inspectobot/rosrover/install/m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 scale=1 1 1; visual mesh filename=file:///home/johnathan/devel/inspectobot/rosrover/install/m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 scale=0.001 0.001 0.001
- added link rear_left_roller6_link, mass 0.15; collision mesh filename=file:///home/johnathan/devel/inspectobot/rosrover/install/m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 scale=1 1 1; visual mesh filename=file:///home/johnathan/devel/inspectobot/rosrover/install/m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 scale=0.001 0.001 0.001
- added link rear_left_roller7_link, mass 0.15; collision mesh filename=file:///home/johnathan/devel/inspectobot/rosrover/install/m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 scale=1 1 1; visual mesh filename=file:///home/johnathan/devel/inspectobot/rosrover/install/m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 scale=0.001 0.001 0.001
- added link rear_left_roller8_link, mass 0.15; collision mesh filename=file:///home/johnathan/devel/inspectobot/rosrover/install/m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 scale=1 1 1; visual mesh filename=file:///home/johnathan/devel/inspectobot/rosrover/install/m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 scale=0.001 0.001 0.001
- added link rear_left_roller9_link, mass 0.15; collision mesh filename=file:///home/johnathan/devel/inspectobot/rosrover/install/m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 scale=1 1 1; visual mesh filename=file:///home/johnathan/devel/inspectobot/rosrover/install/m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 scale=0.001 0.001 0.001
- added link rear_left_wheel_link, mass 1.0; collision mesh filename=file:///home/johnathan/devel/inspectobot/rosrover/install/m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 scale=-0.001 0.001 0.001; visual mesh filename=file:///home/johnathan/devel/inspectobot/rosrover/install/m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 scale=-0.001 0.001 0.001
- added link rear_right_roller10_link, mass 0.15; collision mesh filename=file:///home/johnathan/devel/inspectobot/rosrover/install/m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 scale=1 1 1; visual mesh filename=file:///home/johnathan/devel/inspectobot/rosrover/install/m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 scale=0.001 0.001 0.001
- added link rear_right_roller11_link, mass 0.15; collision mesh filename=file:///home/johnathan/devel/inspectobot/rosrover/install/m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 scale=1 1 1; visual mesh filename=file:///home/johnathan/devel/inspectobot/rosrover/install/m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 scale=0.001 0.001 0.001
- added link rear_right_roller12_link, mass 0.15; collision mesh filename=file:///home/johnathan/devel/inspectobot/rosrover/install/m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 scale=1 1 1; visual mesh filename=file:///home/johnathan/devel/inspectobot/rosrover/install/m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 scale=0.001 0.001 0.001
- added link rear_right_roller13_link, mass 0.15; collision mesh filename=file:///home/johnathan/devel/inspectobot/rosrover/install/m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 scale=1 1 1; visual mesh filename=file:///home/johnathan/devel/inspectobot/rosrover/install/m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 scale=0.001 0.001 0.001
- added link rear_right_roller14_link, mass 0.15; collision mesh filename=file:///home/johnathan/devel/inspectobot/rosrover/install/m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 scale=1 1 1; visual mesh filename=file:///home/johnathan/devel/inspectobot/rosrover/install/m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 scale=0.001 0.001 0.001
- added link rear_right_roller15_link, mass 0.15; collision mesh filename=file:///home/johnathan/devel/inspectobot/rosrover/install/m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 scale=1 1 1; visual mesh filename=file:///home/johnathan/devel/inspectobot/rosrover/install/m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 scale=0.001 0.001 0.001
- added link rear_right_roller1_link, mass 0.15; collision mesh filename=file:///home/johnathan/devel/inspectobot/rosrover/install/m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 scale=1 1 1; visual mesh filename=file:///home/johnathan/devel/inspectobot/rosrover/install/m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 scale=0.001 0.001 0.001
- added link rear_right_roller2_link, mass 0.15; collision mesh filename=file:///home/johnathan/devel/inspectobot/rosrover/install/m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 scale=1 1 1; visual mesh filename=file:///home/johnathan/devel/inspectobot/rosrover/install/m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 scale=0.001 0.001 0.001
- added link rear_right_roller3_link, mass 0.15; collision mesh filename=file:///home/johnathan/devel/inspectobot/rosrover/install/m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 scale=1 1 1; visual mesh filename=file:///home/johnathan/devel/inspectobot/rosrover/install/m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 scale=0.001 0.001 0.001
- added link rear_right_roller4_link, mass 0.15; collision mesh filename=file:///home/johnathan/devel/inspectobot/rosrover/install/m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 scale=1 1 1; visual mesh filename=file:///home/johnathan/devel/inspectobot/rosrover/install/m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 scale=0.001 0.001 0.001
- added link rear_right_roller5_link, mass 0.15; collision mesh filename=file:///home/johnathan/devel/inspectobot/rosrover/install/m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 scale=1 1 1; visual mesh filename=file:///home/johnathan/devel/inspectobot/rosrover/install/m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 scale=0.001 0.001 0.001
- added link rear_right_roller6_link, mass 0.15; collision mesh filename=file:///home/johnathan/devel/inspectobot/rosrover/install/m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 scale=1 1 1; visual mesh filename=file:///home/johnathan/devel/inspectobot/rosrover/install/m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 scale=0.001 0.001 0.001
- added link rear_right_roller7_link, mass 0.15; collision mesh filename=file:///home/johnathan/devel/inspectobot/rosrover/install/m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 scale=1 1 1; visual mesh filename=file:///home/johnathan/devel/inspectobot/rosrover/install/m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 scale=0.001 0.001 0.001
- added link rear_right_roller8_link, mass 0.15; collision mesh filename=file:///home/johnathan/devel/inspectobot/rosrover/install/m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 scale=1 1 1; visual mesh filename=file:///home/johnathan/devel/inspectobot/rosrover/install/m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 scale=0.001 0.001 0.001
- added link rear_right_roller9_link, mass 0.15; collision mesh filename=file:///home/johnathan/devel/inspectobot/rosrover/install/m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 scale=1 1 1; visual mesh filename=file:///home/johnathan/devel/inspectobot/rosrover/install/m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 scale=0.001 0.001 0.001
- added link rear_right_wheel_link, mass 1.0; collision mesh filename=file:///home/johnathan/devel/inspectobot/rosrover/install/m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 scale=0.001 0.001 0.001; visual mesh filename=file:///home/johnathan/devel/inspectobot/rosrover/install/m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 scale=0.001 0.001 0.001
- link front_left_roller10_link: mass 0.3 -> 0.15
- link front_left_roller11_link: mass 0.3 -> 0.15
- link front_left_roller12_link: mass 0.3 -> 0.15
- link front_left_roller13_link: mass 0.3 -> 0.15
- link front_left_roller14_link: mass 0.3 -> 0.15
- link front_left_roller15_link: mass 0.3 -> 0.15
- link front_left_roller1_link: mass 0.3 -> 0.15
- link front_left_roller2_link: mass 0.3 -> 0.15
- link front_left_roller3_link: mass 0.3 -> 0.15
- link front_left_roller4_link: mass 0.3 -> 0.15
- link front_left_roller5_link: mass 0.3 -> 0.15
- link front_left_roller6_link: mass 0.3 -> 0.15
- link front_left_roller7_link: mass 0.3 -> 0.15
- link front_left_roller8_link: mass 0.3 -> 0.15
- link front_left_roller9_link: mass 0.3 -> 0.15
- link front_left_wheel_link: mass 2.0 -> 1.0
Joints:
- added joint front_right_roller10_joint: type continuous, parent front_right_wheel_link, child front_right_roller10_link, origin xyz=0 -0.0362035104982789 -0.02630339004008817 rpy=-0.7989541677433551 -0.6090169187607924 -0.5313896516603533
- added joint front_right_roller11_joint: type continuous, parent front_right_wheel_link, child front_right_roller11_link, origin xyz=0 -0.02237500000000002 -0.038754636819353615 rpy=-1.1831996401397156 -0.3613671239067081 -0.7137243789447655
- added joint front_right_roller12_joint: type continuous, parent front_right_wheel_link, child front_right_roller12_link, origin xyz=0 -0.004677648731227488 -0.044504854817730234 rpy=-1.4966127917301506 -0.07398025001120935 -0.7826515949744619
- added joint front_right_roller13_joint: type continuous, parent front_right_wheel_link, child front_right_roller13_link, origin xyz=0 0.013828510498278887 -0.04255977910420812 rpy=1.3449626171032882 0.22028527385474703 -0.7603177925108144
- added joint front_right_roller14_joint: type continuous, parent front_right_wheel_link, child front_right_roller14_link, origin xyz=0 0.029943594634558885 -0.03325573094011341 rpy=1.0038406803226874 0.4928592704898482 -0.6390993414905143
- added joint front_right_roller15_joint: type continuous, parent front_right_wheel_link, child front_right_roller15_link, origin xyz=0 0.04088115922950639 -0.018201464777642055 rpy=0.5619350361043127 0.7022987807291682 -0.38630030387691144
- added joint front_right_roller1_joint: type continuous, parent front_right_wheel_link, child front_right_roller1_link, origin xyz=0 0.04475 0.0 rpy=-0.0 0.7853981633974482 0.0
- added joint front_right_roller2_joint: type continuous, parent front_right_wheel_link, child front_right_roller2_link, origin xyz=0 0.040881159229506386 0.01820146477764206 rpy=-0.5619350361043128 0.702298780729168 0.3863003038769115
- added joint front_right_roller3_joint: type continuous, parent front_right_wheel_link, child front_right_roller3_link, origin xyz=0 0.029943594634558906 0.033255730940113394 rpy=-1.0038406803226867 0.4928592704898485 0.6390993414905141
- added joint front_right_roller4_joint: type continuous, parent front_right_wheel_link, child front_right_roller4_link, origin xyz=0 0.013828510498278898 0.04255977910420812 rpy=-1.3449626171032882 0.2202852738547472 0.7603177925108144
- added joint front_right_roller5_joint: type continuous, parent front_right_wheel_link, child front_right_roller5_link, origin xyz=0 -0.0046776487312274965 0.04450485481773023 rpy=1.4966127917301504 -0.07398025001120949 0.7826515949744619
- added joint front_right_roller6_joint: type continuous, parent front_right_wheel_link, child front_right_roller6_link, origin xyz=0 -0.02237499999999999 0.03875463681935363 rpy=1.1831996401397162 -0.3613671239067076 0.7137243789447657
- added joint front_right_roller7_joint: type continuous, parent front_right_wheel_link, child front_right_roller7_link, origin xyz=0 -0.03620351049827889 0.026303390040088175 rpy=0.7989541677433554 -0.6090169187607923 0.5313896516603536
- added joint front_right_roller8_joint: type continuous, parent front_right_wheel_link, child front_right_roller8_link, origin xyz=0 -0.0437721051328378 0.00930404816409473 rpy=0.2920075036845471 -0.7637777909460687 0.20499125187874387
- added joint front_right_roller9_joint: type continuous, parent front_right_wheel_link, child front_right_roller9_link, origin xyz=0 -0.043772105132837795 -0.009304048164094738 rpy=-0.29200750368454736 -0.7637777909460687 -0.20499125187874406
- added joint rear_left_roller10_joint: type continuous, parent rear_left_wheel_link, child rear_left_roller10_link, origin xyz=0 -0.0362035104982789 -0.02630339004008817 rpy=-0.7989541677433551 0.6090169187607924 0.5313896516603533
- added joint rear_left_roller11_joint: type continuous, parent rear_left_wheel_link, child rear_left_roller11_link, origin xyz=0 -0.02237500000000002 -0.038754636819353615 rpy=-1.1831996401397156 0.3613671239067081 0.7137243789447655
- added joint rear_left_roller12_joint: type continuous, parent rear_left_wheel_link, child rear_left_roller12_link, origin xyz=0 -0.004677648731227488 -0.044504854817730234 rpy=-1.4966127917301506 0.07398025001120935 0.7826515949744619
- added joint rear_left_roller13_joint: type continuous, parent rear_left_wheel_link, child rear_left_roller13_link, origin xyz=0 0.013828510498278887 -0.04255977910420812 rpy=1.3449626171032882 -0.22028527385474703 0.7603177925108144
- added joint rear_left_roller14_joint: type continuous, parent rear_left_wheel_link, child rear_left_roller14_link, origin xyz=0 0.029943594634558885 -0.03325573094011341 rpy=1.0038406803226874 -0.4928592704898482 0.6390993414905143
- added joint rear_left_roller15_joint: type continuous, parent rear_left_wheel_link, child rear_left_roller15_link, origin xyz=0 0.04088115922950639 -0.018201464777642055 rpy=0.5619350361043127 -0.7022987807291682 0.38630030387691144
- added joint rear_left_roller1_joint: type continuous, parent rear_left_wheel_link, child rear_left_roller1_link, origin xyz=0 0.04475 0.0 rpy=-0.0 -0.7853981633974482 -0.0
- added joint rear_left_roller2_joint: type continuous, parent rear_left_wheel_link, child rear_left_roller2_link, origin xyz=0 0.040881159229506386 0.01820146477764206 rpy=-0.5619350361043128 -0.702298780729168 -0.3863003038769115
- added joint rear_left_roller3_joint: type continuous, parent rear_left_wheel_link, child rear_left_roller3_link, origin xyz=0 0.029943594634558906 0.033255730940113394 rpy=-1.0038406803226867 -0.4928592704898485 -0.6390993414905141
- added joint rear_left_roller4_joint: type continuous, parent rear_left_wheel_link, child rear_left_roller4_link, origin xyz=0 0.013828510498278898 0.04255977910420812 rpy=-1.3449626171032882 -0.2202852738547472 -0.7603177925108144
- added joint rear_left_roller5_joint: type continuous, parent rear_left_wheel_link, child rear_left_roller5_link, origin xyz=0 -0.0046776487312274965 0.04450485481773023 rpy=1.4966127917301504 0.07398025001120949 -0.7826515949744619
- added joint rear_left_roller6_joint: type continuous, parent rear_left_wheel_link, child rear_left_roller6_link, origin xyz=0 -0.02237499999999999 0.03875463681935363 rpy=1.1831996401397162 0.3613671239067076 -0.7137243789447657
- added joint rear_left_roller7_joint: type continuous, parent rear_left_wheel_link, child rear_left_roller7_link, origin xyz=0 -0.03620351049827889 0.026303390040088175 rpy=0.7989541677433554 0.6090169187607923 -0.5313896516603536
- added joint rear_left_roller8_joint: type continuous, parent rear_left_wheel_link, child rear_left_roller8_link, origin xyz=0 -0.0437721051328378 0.00930404816409473 rpy=0.2920075036845471 0.7637777909460687 -0.20499125187874387
- added joint rear_left_roller9_joint: type continuous, parent rear_left_wheel_link, child rear_left_roller9_link, origin xyz=0 -0.043772105132837795 -0.009304048164094738 rpy=-0.29200750368454736 0.7637777909460687 0.20499125187874406
- added joint rear_right_roller10_joint: type continuous, parent rear_right_wheel_link, child rear_right_roller10_link, origin xyz=0 -0.0362035104982789 -0.02630339004008817 rpy=-0.7989541677433551 -0.6090169187607924 -0.5313896516603533
- added joint rear_right_roller11_joint: type continuous, parent rear_right_wheel_link, child rear_right_roller11_link, origin xyz=0 -0.02237500000000002 -0.038754636819353615 rpy=-1.1831996401397156 -0.3613671239067081 -0.7137243789447655
- added joint rear_right_roller12_joint: type continuous, parent rear_right_wheel_link, child rear_right_roller12_link, origin xyz=0 -0.004677648731227488 -0.044504854817730234 rpy=-1.4966127917301506 -0.07398025001120935 -0.7826515949744619
- added joint rear_right_roller13_joint: type continuous, parent rear_right_wheel_link, child rear_right_roller13_link, origin xyz=0 0.013828510498278887 -0.04255977910420812 rpy=1.3449626171032882 0.22028527385474703 -0.7603177925108144
- added joint rear_right_roller14_joint: type continuous, parent rear_right_wheel_link, child rear_right_roller14_link, origin xyz=0 0.029943594634558885 -0.03325573094011341 rpy=1.0038406803226874 0.4928592704898482 -0.6390993414905143
- added joint rear_right_roller15_joint: type continuous, parent rear_right_wheel_link, child rear_right_roller15_link, origin xyz=0 0.04088115922950639 -0.018201464777642055 rpy=0.5619350361043127 0.7022987807291682 -0.38630030387691144
- added joint rear_right_roller1_joint: type continuous, parent rear_right_wheel_link, child rear_right_roller1_link, origin xyz=0 0.04475 0.0 rpy=-0.0 0.7853981633974482 0.0
- added joint rear_right_roller2_joint: type continuous, parent rear_right_wheel_link, child rear_right_roller2_link, origin xyz=0 0.040881159229506386 0.01820146477764206 rpy=-0.5619350361043128 0.702298780729168 0.3863003038769115
- added joint rear_right_roller3_joint: type continuous, parent rear_right_wheel_link, child rear_right_roller3_link, origin xyz=0 0.029943594634558906 0.033255730940113394 rpy=-1.0038406803226867 0.4928592704898485 0.6390993414905141
- added joint rear_right_roller4_joint: type continuous, parent rear_right_wheel_link, child rear_right_roller4_link, origin xyz=0 0.013828510498278898 0.04255977910420812 rpy=-1.3449626171032882 0.2202852738547472 0.7603177925108144
- added joint rear_right_roller5_joint: type continuous, parent rear_right_wheel_link, child rear_right_roller5_link, origin xyz=0 -0.0046776487312274965 0.04450485481773023 rpy=1.4966127917301504 -0.07398025001120949 0.7826515949744619
- added joint rear_right_roller6_joint: type continuous, parent rear_right_wheel_link, child rear_right_roller6_link, origin xyz=0 -0.02237499999999999 0.03875463681935363 rpy=1.1831996401397162 -0.3613671239067076 0.7137243789447657
- added joint rear_right_roller7_joint: type continuous, parent rear_right_wheel_link, child rear_right_roller7_link, origin xyz=0 -0.03620351049827889 0.026303390040088175 rpy=0.7989541677433554 -0.6090169187607923 0.5313896516603536
- added joint rear_right_roller8_joint: type continuous, parent rear_right_wheel_link, child rear_right_roller8_link, origin xyz=0 -0.0437721051328378 0.00930404816409473 rpy=0.2920075036845471 -0.7637777909460687 0.20499125187874387
- added joint rear_right_roller9_joint: type continuous, parent rear_right_wheel_link, child rear_right_roller9_link, origin xyz=0 -0.043772105132837795 -0.009304048164094738 rpy=-0.29200750368454736 -0.7637777909460687 -0.20499125187874406
- joint wheel2_wheel_joint: child wheel2 -> front_right_wheel_link
- joint wheel3_wheel_joint: child wheel3 -> rear_right_wheel_link
- joint wheel4_wheel_joint: child wheel4 -> rear_left_wheel_link
